File: subs/body/body.sch (KiCad schematic (older format))
At the start: 74 parts, among them IC1 ATMEGA328P(B), P1 CON_BAT_IN, P3 CON_POLOLU_PWR2, P4 CONN_BREAKOUT4, P5 CONN_BREAKOUT2, P6 CONN_BREAKOUT3, P7 CONN_BREAKOUT5, P8 CON_BAT_OUT, Q1 CSD25402Q3A, Q2 CSD25402Q3A, Q3 CSD25402Q3A, Q4 CSD25402Q3A, Q5 CSD25402Q3A, Q6 CSD25402Q3A, SW1 SPST_Small, SW2 SPST_Small, U1 LTC4412, U10 74LVC2G07, U11 74LVC2G07, U12 LTC4412, U2 LTC4412, U3 DRV8834-SSOP, U4 TMP36GRT, U5 LTC4412, U6 RT9715GGB, 0.7A, U7 RT9715GGB, 0.7A, U8 RT9715GGB, 0.7A, U9 RT9715GGB, 0.7A, Y1 16MHz

Commit message: Before major layout change
Parts:
- removed C13: 100nF, Capacitors_SMD:C_0402, symbol C_Small
- removed U4: TMP36GRT, TO_SOT_Packages_SMD:SOT-23-5_Handsoldering, symbol TMP36
- P4: value CONN_BREAKOUT4 -> CONN3
- P5: value CONN_BREAKOUT2 -> CONN1; footprint Socket_Strips:Socket_Strip_Straight_1x12_Pitch1.27mm -> Socket_Strips:Socket_Strip_Straight_1x15_Pitch1.27mm; symbol CONN_01X12 -> CONN_01X15
- P6: value CONN_BREAKOUT3 -> CONN2
- P7: value CONN_BREAKOUT5 -> CONN4
Connections:
- net labels added: A6, BAT_PATH1, BAT_PATH2
- net labels removed: TMP
- wire segments 276 -> 389
Other:
- moved on the sheet: P4, P6

Commit message: Finished routing of body board
Parts:
- removed C12: 10uF, Capacitors_SMD:C_0805, symbol C_Small
- removed C26, C27: 100nF, Capacitors_SMD:C_0402, symbol C_Small
- removed P3: CON_POLOLU_PWR2, Misc:Pololu-5V-2.54-U3V50F5, symbol CON_POLOLU_PWR2
- removed P8: CON_BAT_OUT, Pin_Headers:Pin_Header_Straight_2x04, symbol CONN_02X04
- removed Q5, Q6: CSD25402Q3A, Housings_DFN_QFN:DFN-8-MOS_3x3mm_Pitch0.65mm, symbol CSD25402Q3A
- removed SW1, SW2: SPST_Small, Buttons_Switches_SMD:MTA2_4.5x2.3mm, symbol SPST_Small
- removed U1, U12, U5: LTC4412, TO_SOT_Packages_SMD:SOT-23-6_Handsoldering, symbol LTC4412
- added C13, C32, C41: 100nF, Capacitors_SMD:C_0402, symbol C_Small
- added C33, C34: 1uF, Capacitors_SMD:C_0402, symbol C_Small
- added C35, C37: 4.7nF, Capacitors_SMD:C_0402, symbol C_Small
- added D1, D2, D3, D4: ESB5B5.0S, Diodes_SMD:SOD-523, symbol TVS_Small
- added IC2: ATMEGA328P(B), Housings_QFP:TQFP-32_7x7mm_Pitch0.8mm, symbol ARDUINO-ATMEGA328P(B)
- added L2: 4.7uH, Capacitors_SMD:C_0603, symbol L_Small
- added P10: BAT2+, Pin_Headers:Pin_Header_Straight_1x01, symbol CONN_01X01
- added P11, P9: BAT1-, Pin_Headers:Pin_Header_Straight_1x01, symbol CONN_01X01
- added P12: CONN_RESET, Pin_Headers:Pin_Header_Straight_1x02_Pitch1.27mm, symbol CONN_01X02
- added P2: CONN_VCC, Pin_Headers:Pin_Header_Straight_1x02, symbol CONN_01X02
- added P8: BAT1+, Pin_Headers:Pin_Header_Straight_1x01, symbol CONN_01X01
- added Q10, Q7, Q8, Q9: CSD16327Q3, Housings_DFN_QFN:DFN-8-MOS_3x3mm_Pitch0.65mm, symbol CSD16325Q5
- added Q11, Q12, Q13, Q14: CSD25404Q3A, Housings_DFN_QFN:DFN-8-MOS_3x3mm_Pitch0.65mm, symbol CSD25402Q3A
- added Q5, Q6: MTM231232LBF, TO_SOT_Packages_SMD:SC-70, symbol Q_PMOS_WITH_DIODE_GSD
- added R11, R20, R21, R25, R27, R8: 5M, Resistors_SMD:R_0402, symbol R_Small
- added R12, R13: 330, Resistors_SMD:R_0402, symbol R_Small
- added R2, R28, R29, R3, R32, R33: 10K, Resistors_SMD:R_0402, symbol R_Small
- added R22, R23: 2.2K, Resistors_SMD:R_0402, symbol R_Small
- added R24, R26: 2M, Resistors_SMD:R_0402, symbol R_Small
- added R30, R31: 100, Resistors_SMD:R_0402, symbol R_Small
- added SW1, SW2: SW_PUSH_Small_Horizontal, Buttons_Switches_SMD:MTA2_4.5x2.3mm, symbol SW_PUSH_Small_Horizontal
- added U1: 74LVC2G07, TO_SOT_Packages_SMD:SC-70-6, symbol 74LVC2G07
- added U12: TMP101, TO_SOT_Packages_SMD:SOT-23-6, symbol TMP10X
- added U13, U5: bq29700, Housings_DFN_QFN:DFN-6-1.5x1.5mm_Pitch0.5mm, symbol bq297xx
- added U14, U15, U4: LTC4412, TO_SOT_Packages_SMD:SOT-23-6, symbol LTC4412
- added Y2: 16MHz, Crystals:Resonator_3x1.3mm, symbol CRYSTAL_SMD
- C1: footprint Capacitors_SMD:C_0805 -> Capacitors_SMD:C_0603
- C18: footprint Capacitors_SMD:C_0402 -> Capacitors_SMD:C_0805
- C24, C25: value 100nF -> 100pF
- C5: value 1uF -> 10uF
- C6: value 1uF -> 100nF; footprint Capacitors_SMD:C_0603 -> Capacitors_SMD:C_0402
- C7, C8: value 22uF -> 100nF; footprint Capacitors_SMD:C_0805 -> Capacitors_SMD:C_0402
- L1: value 10uH -> 4.7uH
- P1: value CON_BAT_IN -> CONN5
- P4: footprint Socket_Strips:Socket_Strip_Straight_1x10_Pitch1.27mm -> Socket_Strips:Socket_Strip_Straight_1x06_Pitch1.27mm; symbol CONN_01X10 -> CONN_01X06
- P5, P6: footprint Socket_Strips:Socket_Strip_Straight_1x15_Pitch1.27mm -> Socket_Strips:Socket_Strip_Straight_1x12_Pitch1.27mm; symbol CONN_01X15 -> CONN_01X12
- P7: footprint Socket_Strips:Socket_Strip_Straight_1x05_Pitch1.27mm -> Pin_Headers:Pin_Header_Straight_1x09_Pitch1.27mm; symbol CONN_01X05 -> CONN_01X09
- Q1, Q2, Q3, Q4: value CSD25402Q3A -> CSD25404Q3A
- R1, R10, R14, R15, R16, R17, R18, R19, R7, R9: footprint Resistors_SMD:R_0402_Handsoldering -> Resistors_SMD:R_0402
- R4: value 1K -> 10K; footprint Resistors_SMD:R_0402_Handsoldering -> Resistors_SMD:R_0402
- R5: value 10K -> 1K; footprint Resistors_SMD:R_0402_Handsoldering -> Resistors_SMD:R_0402
- R6: value 10K -> 100K; footprint Resistors_SMD:R_0402_Handsoldering -> Resistors_SMD:R_0402
- U10, U11: footprint TO_SOT_Packages_SMD:SC-70-6_Handsoldering -> TO_SOT_Packages_SMD:SC-70-6
- U2: footprint TO_SOT_Packages_SMD:SOT-23-6_Handsoldering -> TO_SOT_Packages_SMD:SOT-23-6
- U6, U7, U8, U9: footprint TO_SOT_Packages_SMD:SOT-23-5_Handsoldering -> TO_SOT_Packages_SMD:SOT-23-5
Connections:
- net BAT_CTL1 is gone; now on net SRV_CAM: IC1.11 ((AIN1/PD7)D7)
- net BAT_STAT1 is gone; now on net IR_TX: P7.4 (P4)
- net BAT: now also P1.3 (P3), P1.4 (P4), P1.5 (P5), P1.6 (P6), Q13.1 (S), Q13.2 (S), Q13.3 (S), Q14.1 (S), Q14.2 (S), Q14.3 (S), R31.2, U14.6 (SENSE), U15.6 (SENSE); no longer C21.2, C7.2, C8.2, Q3.1 (S), Q3.2 (S), Q3.3 (S), Q4.1 (S), Q4.2 (S), Q4.3 (S), U2.6 (SENSE), U9.5 (VIN)
- net BAT_INT: now also P7.5 (P5), R5.2; no longer P5.6 (P6), R4.2
- net CHARGE: now also C11.1, P1.7 (P7), Q1.1 (S), Q1.2 (S), Q1.3 (S), Q2.1 (S), Q2.2 (S), Q2.3 (S), U2.1 (VIN), C41.2, R30.2, U4.1 (VIN); no longer C14.1, P1.4 (P4)
- net EP_EN: now also IC2.25 ((ADC2/PC2)A2); no longer P7.3 (P3)
- net EP_TXD: now also P5.3 (P3); no longer P5.4 (P4)
- net EP_VCC: now also P4.5 (P5), P4.6 (P6); no longer C25.2, P4.10 (P10), P4.9 (P9)
- net FAN_EN: now also IC1.2 ((XCK/T0/PD4)D4); no longer P6.4 (P4)
- net FAN_PWM: now also IC1.32 ((OC3B/OC4B/INT0/PD2)D2), P6.4 (P4); no longer IC1.15 ((OC2A/TXD1/MOSI/PB3)D11), P6.6 (P6)
- net FAN_VOUT: now also P6.2 (P2); no longer P6.5 (P5)
- net GND: now also C10.1, C24.2, C25.2, C7.2, C8.2, P1.1 (P1), P1.10 (P10), P1.2 (P2), P1.9 (P9), C32.1, C33.2, C34.2, C35.2, C37.2, C41.1, D1.2, D2.2, D3.2, D4.2, IC2.21 (GND), IC2.5 (GND), P2.1 (P1), Q10.1 (S), Q10.2 (S), Q10.3 (S), Q9.1 (S), Q9.2 (S), Q9.3 (S), R20.2, R21.2, R22.1, R23.1, R24.2, R25.2, R26.2, R27.2, SW1.2, SW2.1, U1.2 (GND), U1.2 (GND), U12.2 (GND), U14.2 (GND), U15.2 (GND), U4.2 (GND), Y2.3 (case); no longer C10.2, C14.2, C24.1, C25.1, C7.1, C8.1, P1.5 (P5), P1.6 (P6), P4.5 (P5), P4.6 (P6), P5.12 (P12), P5.15 (P15), P5.7 (P7), P6.12 (P12), P6.7 (P7)
- net IR_RX: now also P7.6 (P6), IC2.2 ((XCK/T0/PD4)D4); no longer IC1.2 ((XCK/T0/PD4)D4), P6.8 (P8)
- net IR_TX: now also IC2.32 ((OC3B/OC4B/INT0/PD2)D2); no longer IC1.32 ((OC3B/OC4B/INT0/PD2)D2), P6.9 (P9)
- net LED_CLK: now also P6.11 (P11); no longer P6.14 (P14)
- net LED_DAT: now also P6.10 (P10); no longer P6.13 (P13)
- net LED_EN: now also IC1.23 ((MISO1/ADC0/PC0)A0); no longer P5.5 (P5)
- net LED_VOUT: now also P6.12 (P12); no longer C24.2, P6.15 (P15)
- net SRV_BRAKE: now also IC1.13 ((OC1A/PB1)D9), P5.7 (P7); no longer IC1.16 ((RXD1/MISO/PB4)D12), P5.10 (P10)
- net SRV_CAM: now also P5.5 (P5); no longer IC1.13 ((OC1A/PB1)D9), P5.8 (P8)
- net SRV_EN: now also IC1.19 ((~SS1~/ADC6/PE2)A6); no longer P6.1 (P1)
- net SRV_FOOT: now also IC1.12 ((CLKO/ICP1/PB0)D8), P5.6 (P6); no longer IC1.14 ((OC1B/~SS~/PB2)D10), P5.9 (P9)
- net SRV_LOCK: now also IC1.14 ((OC1B/~SS~/PB2)D10), P5.8 (P8); no longer IC1.17 ((PCINT5/SCK/PB5)D13), P5.11 (P11)
- net SRV_VOUT: now also P5.12 (P12); no longer P6.2 (P2)
- net STEP_DIR: now also IC1.10 ((OC0A/AIN0/PD6)D6); no longer P7.1 (P1)
- net UART_RX: now also P5.4 (P4), U1.1; no longer P5.3 (P3)
- net UART_TX: now also U1.4
- net VCC: now also C10.2, C21.2, C5.1, C6.1, R4.2, R6.2, U9.5 (VIN), C32.2, IC2.4 (VCC), L2.1, P2.2 (P2), R2.1, R3.1, R32.1, R33.1, U1.5 (VCC), U1.5 (VCC), U12.4 (V+); no longer P4.7 (P7), P4.8 (P8)
- net ~STEP_SLP: now also IC2.26 ((ADC3/PC3)A3); no longer P7.2 (P2)
- net at Q1.4 (G), Q3.4 (G): now also U2.5 (GATE)
- net at Q2.4 (G), Q4.4 (G): now also U4.5 (GATE); no longer U2.5 (GATE)
- removed net A0: IC1.23 ((MISO1/ADC0/PC0)A0), P5.14 (P14)
- removed net A6: IC1.19 ((~SS1~/ADC6/PE2)A6), P5.13 (P13)
- net BAT_CTL2 renamed CHG1_CTL
- net CHG1_CTL: now also IC2.12 ((CLKO/ICP1/PB0)D8); no longer IC1.10 ((OC0A/AIN0/PD6)D6)
- net BAT_PATH1 renamed CHG1_PATH2
- net BAT_PATH2 renamed CHG2_PATH2
- net BAT_STAT2 renamed CHG1_STAT
- net CHG1_STAT: now also IC2.13 ((OC1A/PB1)D9); no longer P7.5 (P5)
- removed net BAT_VIN1: C5.1, P1.10 (P10), P1.7 (P7), P1.9 (P9), Q1.1 (S), Q1.2 (S), Q1.3 (S), R5.2
- removed net BAT_VIN2: C6.1, P1.1 (P1), P1.2 (P2), P1.3 (P3), Q2.1 (S), Q2.2 (S), Q2.3 (S), R6.2, U2.1 (VIN)
- removed net BAT_VOLT1: C10.1, IC1.25 ((ADC2/PC2)A2), R5.1
- removed net BAT_VOLT2: C11.1, IC1.26 ((ADC3/PC3)A3), R6.1
- net CHG_STAT1 renamed TMP_INT0
- net TMP_INT0: now also U12.3 (ALERT/ADD1)
- net CHG_STAT2 renamed PE0
- net PE0: now also P6.1 (P1)
- net INT renamed FAN_TACHO
- net RESET renamed ~RESET0
- net ~RESET0: now also P6.5 (P5)
- net RXD renamed RXD0
- net RXD0: now also U1.6; no longer U11.4
- net SCL renamed SCL0
- net SCL0: now also P6.6 (P6), R2.2, U12.1 (SCL); no longer P6.10 (P10)
- net SDA renamed SDA0
- net SDA0: now also P6.7 (P7), R3.2, U12.6 (SDA); no longer P6.11 (P11)
- net TXD renamed TXD0
- net TXD0: now also U1.3; no longer U11.1
- new net: Q12.4 (G), Q14.4 (G), U15.5 (GATE)
- new net: Q11.4 (G), Q13.4 (G), U14.5 (GATE)
- new net: Q7.4 (G), R8.2, U5.3 (DOUT)
- new net: R22.2, U5.6 (V-)
- new net: C13.2, R12.2, U5.5 (BAT)
- new net: Q5.2 (S), R12.1
- new net: Q8.4 (G), R11.2, U13.3 (DOUT)
- new net: R23.2, U13.6 (V-)
- new net: C14.2, R13.2, U13.5 (BAT)
- new net: Q6.2 (S), R13.1
- new net: C7.1, IC2.18 (AVCC), L2.2
- new net: C8.1, IC2.20 (AREF)
- new net: C9.1, IC2.1 ((OC2B/INT1/PD3)D3), R5.1
- new net: IC2.7 (XTAL1(PB6/TOSC1)), Y2.1
- new net: IC2.8 (XTAL2(PB7/TOSC2)), Y2.2
- new net A2: IC1.25 ((ADC2/PC2)A2), P6.9 (P9)
- new net BAT1+: C33.1, P8.1 (P1), Q11.1 (S), Q11.2 (S), Q11.3 (S), Q3.1 (S), Q3.2 (S), Q3.3 (S), Q5.3 (D), R28.2, U14.1 (VIN), U2.6 (SENSE)
- new net BAT1-: C13.1, P9.1 (P1), Q5.1 (G), Q7.1 (S), Q7.2 (S), Q7.3 (S), R8.1, U5.4 (VSS)
- new net BAT1_CTL: IC2.9 ((OC0B/T1/PD5)D5), U14.3 (CTL)
- new net BAT1_PATH: Q7.5 (D), Q7.6 (D), Q7.7 (D), Q7.8 (D), Q9.5 (D), Q9.6 (D), Q9.7 (D), Q9.8 (D)
- new net BAT1_PATH2: Q11.5 (D), Q11.6 (D), Q11.7 (D), Q11.8 (D), Q13.5 (D), Q13.6 (D), Q13.7 (D), Q13.8 (D)
- new net BAT1_STAT: IC2.10 ((OC0A/AIN0/PD6)D6), U14.4 (STAT)
- new net BAT2+: C34.1, P10.1 (P1), Q12.1 (S), Q12.2 (S), Q12.3 (S), Q4.1 (S), Q4.2 (S), Q4.3 (S), Q6.3 (D), R29.2, U15.1 (VIN), U4.6 (SENSE)
- new net BAT2-: C14.1, P11.1 (P1), Q6.1 (G), Q8.1 (S), Q8.2 (S), Q8.3 (S), R11.1, U13.4 (VSS)
- new net BAT2_CTL: IC2.17 ((PCINT5/SCK/PB5)D13), U15.3 (CTL)
- new net BAT2_PATH: Q10.5 (D), Q10.6 (D), Q10.7 (D), Q10.8 (D), Q8.5 (D), Q8.6 (D), Q8.7 (D), Q8.8 (D)
- new net BAT2_PATH2: Q12.5 (D), Q12.6 (D), Q12.7 (D), Q12.8 (D), Q14.5 (D), Q14.6 (D), Q14.7 (D), Q14.8 (D)
- new net BAT2_STAT: IC2.14 ((OC1B/~SS~/PB2)D10), U15.4 (STAT)
- new net BUTTON: IC1.26 ((ADC3/PC3)A3), P6.8 (P8)
- new net CHG2_CTL: IC2.15 ((OC2A/TXD1/MOSI/PB3)D11), U4.3 (CTL)
- new net CHG2_STAT: IC2.16 ((RXD1/MISO/PB4)D12), U4.4 (STAT)
- new net COUT1: Q9.4 (G), R20.1, U5.2 (COUT)
- new net COUT2: Q10.4 (G), R21.1, U13.2 (COUT)
- new net FRAME_STOP: IC1.17 ((PCINT5/SCK/PB5)D13), P5.11 (P11)
- new net HOST_INT: IC2.6 (PE1(SCL1/T4)(VCC)), P7.8 (P8)
- new net PWR_INT: IC2.3 (PE0(SDA1/ACO)(GND)), P7.7 (P7)
- new net RXD1: IC2.30 ((OC3A/PD0)RXD), R6.1, U11.4
- new net SCL1: IC2.28 ((SCL/ADC5/PC5)A5), P7.2 (P2), R33.2
- new net SDA1: IC2.27 ((SDA/ADC4/PC4)A4), P7.1 (P1), R32.2
- new net STEP_STOP1: IC1.15 ((OC2A/TXD1/MOSI/PB3)D11), P5.9 (P9)
- new net STEP_STOP2: IC1.16 ((RXD1/MISO/PB4)D12), P5.10 (P10)
- new net TMP_INT1: IC2.11 ((AIN1/PD7)D7), P7.9 (P9)
- new net TXD1: IC2.31 ((OC4A/PD1)TXD), U11.1
- new net VBAT: C25.1, D4.1, IC2.22 ((MOSI1/ADC7/PE3)A7), R27.1, R31.1
- new net VBAT1: C35.1, D2.1, IC2.23 ((MISO1/ADC0/PC0)A0), R24.1, R28.1
- new net VBAT2: C37.1, D3.1, IC2.24 ((SCK1/ADC1/PC1)A1), R26.1, R29.1
- new net VCHG: C24.1, D1.1, IC2.19 ((~SS1~/ADC6/PE2)A6), R25.1, R30.1
- new net ~EXT_RST1: P12.1 (P1), SW1.1
- new net ~EXT_RST2: P12.2 (P2), SW2.2
- new net ~RESET1: IC2.29 (~RESET~(PC6)), P7.3 (P3), R4.1
- no-connect marks 5 -> 6
Other:
- note added: "Battery Protector"
- note added: "Charge Balancer"
- note added: "Due to space\nconstraint, \nthese output \ncapacitors are\nrelocated on\non power \nboard"
- note added: "Load Balancer"
- note added: "Reverse protection for bq2970. \nYes, the protector IC itself needs\nprotection, too. By blocking \nreverse connection here, we \neffectively prevents reverse \nconduction on the main BAT \npath. The bonus here is that \nwe can use a much cheaper \nMOSFET."
- note removed: "Optional charger balancer"
- moved on the sheet: C1, C15, C16, C17, C18, C19, C2, C20, C21, C22, C23, C28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

Commit message: In progress, commit for backup
Parts:
- removed P12: CONN_RESET, Pin_Headers:Pin_Header_Straight_1x02_Pitch1.27mm, symbol CONN_01X02
- removed U12: TMP101, TO_SOT_Packages_SMD:SOT-23-6, symbol TMP10X
- added U12: MCP9808, Housings_DFN_QFN:DFN-8-1EP_3x2mm_Pitch0.5mm, symbol MCP9808
- P4: footprint Socket_Strips:Socket_Strip_Straight_1x06_Pitch1.27mm -> Pin_Headers:Pin_Header_Straight_1x06_Pitch1.27mm
- P5: footprint Socket_Strips:Socket_Strip_Straight_1x12_Pitch1.27mm -> Pin_Headers:Pin_Header_Straight_1x12_Pitch1.27mm
- P6: footprint Socket_Strips:Socket_Strip_Straight_1x12_Pitch1.27mm -> Pin_Headers:Pin_Header_Straight_1x15_Pitch1.27mm; symbol CONN_01X12 -> CONN_01X15
- Q1, Q11, Q12, Q13, Q14, Q2, Q3, Q4: value CSD25404Q3A -> AON7423; symbol CSD25402Q3A -> AON7423
- Q10, Q7, Q8, Q9: value CSD16327Q3 -> CSD16327Q3/AON7524
Connections:
- net ~EXT_RST1 is gone; now on net GND: SW1.1
- net ~EXT_RST2 is gone; now on net ~RESET1: SW2.2
- net A2: now also P6.12 (P12); no longer P6.9 (P9)
- net BAT: now also Q13.5 (D), Q13.6 (D), Q13.7 (D), Q13.8 (D), Q14.5 (D), Q14.6 (D), Q14.7 (D), Q14.8 (D); no longer Q13.1 (S), Q13.2 (S), Q13.3 (S), Q14.1 (S), Q14.2 (S), Q14.3 (S)
- net BAT1+: now also Q11.5 (D), Q11.6 (D), Q11.7 (D), Q11.8 (D), Q3.5 (D), Q3.6 (D), Q3.7 (D), Q3.8 (D); no longer Q11.1 (S), Q11.2 (S), Q11.3 (S), Q3.1 (S), Q3.2 (S), Q3.3 (S)
- net BAT1_PATH2: now also Q11.1 (S), Q11.2 (S), Q11.3 (S), Q13.1 (S), Q13.2 (S), Q13.3 (S); no longer Q11.5 (D), Q11.6 (D), Q11.7 (D), Q11.8 (D), Q13.5 (D), Q13.6 (D), Q13.7 (D), Q13.8 (D)
- net BAT2+: now also Q12.5 (D), Q12.6 (D), Q12.7 (D), Q12.8 (D), Q4.5 (D), Q4.6 (D), Q4.7 (D), Q4.8 (D); no longer Q12.1 (S), Q12.2 (S), Q12.3 (S), Q4.1 (S), Q4.2 (S), Q4.3 (S)
- net BAT2_CTL: now also P6.3 (P3)
- net BAT2_PATH2: now also Q12.1 (S), Q12.2 (S), Q12.3 (S), Q14.1 (S), Q14.2 (S), Q14.3 (S); no longer Q12.5 (D), Q12.6 (D), Q12.7 (D), Q12.8 (D), Q14.5 (D), Q14.6 (D), Q14.7 (D), Q14.8 (D)
- net BUTTON: now also P6.11 (P11); no longer P6.8 (P8)
- net CHARGE: now also Q1.5 (D), Q1.6 (D), Q1.7 (D), Q1.8 (D), Q2.5 (D), Q2.6 (D), Q2.7 (D), Q2.8 (D); no longer Q1.1 (S), Q1.2 (S), Q1.3 (S), Q2.1 (S), Q2.2 (S), Q2.3 (S)
- net CHG1_PATH2: now also Q1.1 (S), Q1.2 (S), Q1.3 (S), Q3.1 (S), Q3.2 (S), Q3.3 (S); no longer Q1.5 (D), Q1.6 (D), Q1.7 (D), Q1.8 (D), Q3.5 (D), Q3.6 (D), Q3.7 (D), Q3.8 (D)
- net CHG2_CTL: now also P6.2 (P2)
- net CHG2_PATH2: now also Q2.1 (S), Q2.2 (S), Q2.3 (S), Q4.1 (S), Q4.2 (S), Q4.3 (S); no longer Q2.5 (D), Q2.6 (D), Q2.7 (D), Q2.8 (D), Q4.5 (D), Q4.6 (D), Q4.7 (D), Q4.8 (D)
- net CHG2_STAT: now also P6.1 (P1)
- net FAN_PWM: now also P6.7 (P7); no longer P6.4 (P4)
- net FAN_TACHO: now also P6.6 (P6); no longer P6.3 (P3)
- net FAN_VOUT: now also P6.5 (P5); no longer P6.2 (P2)
- net FRAME_STOP: now also P5.12 (P12); no longer P5.11 (P11)
- net GND: now also U12.4 (GND), U12.6 (A1), U12.7 (A0), U12.9 (GND); no longer SW1.2
- net HOST_INT: now also IC2.11 ((AIN1/PD7)D7); no longer IC2.6 (PE1(SCL1/T4)(VCC))
- net LED_CLK: now also P6.14 (P14); no longer P6.11 (P11)
- net LED_DAT: now also P6.13 (P13); no longer P6.10 (P10)
- net LED_VOUT: now also P6.15 (P15); no longer P6.12 (P12)
- net SCL0: now also P6.9 (P9), U12.1 (SDA); no longer P6.6 (P6)
- net SDA0: now also P6.10 (P10), U12.2 (SCL); no longer P6.7 (P7)
- net SRV_VOUT: now also P5.9 (P9); no longer P5.12 (P12)
- net TMP_INT0: now also IC1.3 (PE0(SDA1/ACO)(GND)), P6.4 (P4), U12.3 (ALERT); no longer IC1.6 (PE1(SCL1/T4)(VCC))
- net TMP_INT1: now also IC2.6 (PE1(SCL1/T4)(VCC)); no longer IC2.11 ((AIN1/PD7)D7)
- net VBAT1: now also IC2.24 ((SCK1/ADC1/PC1)A1); no longer IC2.23 ((MISO1/ADC0/PC0)A0)
- net VBAT2: now also IC2.19 ((~SS1~/ADC6/PE2)A6); no longer IC2.24 ((SCK1/ADC1/PC1)A1)
- net VCC: now also U12.8 (Vdd)
- net VCHG: now also IC2.23 ((MISO1/ADC0/PC0)A0); no longer IC2.19 ((~SS1~/ADC6/PE2)A6)
- net ~RESET0: now also P6.8 (P8), SW1.2; no longer P6.5 (P5)
- removed net PE0: IC1.3 (PE0(SDA1/ACO)(GND)), P6.1 (P1)
- net STEP_STOP1 renamed MOSI0
- net MOSI0: now also P5.10 (P10); no longer P5.9 (P9)
- net STEP_STOP2 renamed MISO0
- net MISO0: now also P5.11 (P11); no longer P5.10 (P10)
- new net TMP_ADDR: IC1.6 (PE1(SCL1/T4)(VCC)), U12.5 (A2)
- no-connect marks 6 -> 5
Other:
- moved on the sheet: P2, SW1, SW2

Commit message: Major modification of body board and companions
Parts:
- removed C32: 100nF, Capacitors_SMD:C_0402, symbol C_Small
- removed U12: MCP9808, Housings_DFN_QFN:DFN-8-1EP_3x2mm_Pitch0.5mm, symbol MCP9808
- P5: footprint Pin_Headers:Pin_Header_Straight_1x12_Pitch1.27mm -> Pin_Headers:Pin_Header_Straight_1x13_Pitch1.27mm; symbol CONN_01X12 -> CONN_01X13
- Q5, Q6: value MTM231232LBF -> AO3419/AO3401; footprint TO_SOT_Packages_SMD:SC-70 -> TO_SOT_Packages_SMD:SOT-23
- Q7, Q8: value CSD16327Q3/AON7524 -> AON7524/CSD16327Q3
Connections:
- net TMP_ADDR is gone; now on net ~STEP_SLP: IC1.6 (PE1(SCL1/T4)(VCC))
- net A2: now also P5.9 (P9); no longer P6.12 (P12)
- net BAT: no longer Q13.5 (D), Q13.6 (D), Q13.7 (D), Q13.8 (D), Q14.5 (D), Q14.6 (D), Q14.7 (D), Q14.8 (D)
- net BAT2_CTL: now also IC2.14 ((OC1B/~SS~/PB2)D10); no longer IC2.17 ((PCINT5/SCK/PB5)D13)
- net BAT2_STAT: now also IC2.13 ((OC1A/PB1)D9); no longer IC2.14 ((OC1B/~SS~/PB2)D10)
- net BUTTON: now also P6.12 (P12); no longer P6.11 (P11)
- net CHG1_CTL: now also IC2.11 ((AIN1/PD7)D7); no longer IC2.12 ((CLKO/ICP1/PB0)D8)
- net CHG1_STAT: now also IC2.12 ((CLKO/ICP1/PB0)D8); no longer IC2.13 ((OC1A/PB1)D9)
- net FAN_EN: now also IC1.3 (PE0(SDA1/ACO)(GND)); no longer IC1.2 ((XCK/T0/PD4)D4)
- net FAN_PWM: now also IC1.1 ((OC2B/INT1/PD3)D3), P6.6 (P6); no longer IC1.32 ((OC3B/OC4B/INT0/PD2)D2), P6.7 (P7)
- net FAN_TACHO: now also IC1.32 ((OC3B/OC4B/INT0/PD2)D2), P6.8 (P8); no longer IC1.1 ((OC2B/INT1/PD3)D3), P6.6 (P6)
- net FAN_VOUT: now also P6.4 (P4); no longer P6.5 (P5)
- net HOST_INT: now also IC1.2 ((XCK/T0/PD4)D4), P6.7 (P7); no longer IC2.11 ((AIN1/PD7)D7), P7.8 (P8)
- net IR_RX: now also P7.7 (P7); no longer P7.6 (P6)
- net IR_TX: now also IC2.1 ((OC2B/INT1/PD3)D3), P7.6 (P6); no longer IC2.32 ((OC3B/OC4B/INT0/PD2)D2), P7.4 (P4)
- net PWR_INT: now also IC2.26 ((ADC3/PC3)A3), P7.1 (P1); no longer IC2.3 (PE0(SDA1/ACO)(GND)), P7.7 (P7)
- net SCL0: now also P6.10 (P10), R3.2; no longer P6.9 (P9), R2.2
- net SCL1: now also P7.3 (P3); no longer P7.2 (P2)
- net SDA0: now also P6.11 (P11), R2.2; no longer P6.10 (P10), R3.2
- net SDA1: now also P7.2 (P2); no longer P7.1 (P1)
- net SRV_VOUT: now also P5.13 (P13); no longer P5.9 (P9)
- net STEP: now also IC1.10 ((OC0A/AIN0/PD6)D6); no longer IC1.9 ((OC0B/T1/PD5)D5)
- net STEP_DIR: now also IC1.9 ((OC0B/T1/PD5)D5); no longer IC1.10 ((OC0A/AIN0/PD6)D6)
- net ~RESET0: now also P6.9 (P9); no longer P6.8 (P8)
- net ~RESET1: now also P7.4 (P4); no longer P7.3 (P3)
- net ~STEP_SLP: no longer IC2.26 ((ADC3/PC3)A3)
- net at C9.1, R5.1: now also IC2.32 ((OC3B/OC4B/INT0/PD2)D2); no longer IC2.1 ((OC2B/INT1/PD3)D3)
- removed net TMP_INT0: IC1.3 (PE0(SDA1/ACO)(GND)), P6.4 (P4)
- net TMP_INT1 renamed SCL2
- new net: Q14.5 (D), Q14.6 (D), Q14.8 (D)
- new net: Q13.5 (D), Q13.6 (D), Q13.8 (D)
- new net SDA2: IC2.3 (PE0(SDA1/ACO)(GND)), P7.8 (P8)
- new net TMP_INT: IC2.17 ((PCINT5/SCK/PB5)D13), P6.5 (P5)
Other:
- note removed: "Due to space\nconstraint, \nthese output \ncapacitors are\nrelocated on\non power \nboard"
- moved on the sheet: C9, R5
