File: subs/body/breakout/breakout.sch (KiCad schematic (older format))
At the start: 25 parts, among them P1 CONN_SRV_CAM, P10 CONN_UART, P11 CONN_I2C, P12 CONN_FAN, P14 CONN_IR, P15 CONN_STEP, P16 CONN_EP_VCC, P17 CONN_BTN, P18 CONN3, P19 CONN4, P2 CONN_SRV_LOCK, P21 CONN1, P22 CONN2, P3 CONN_SRV_BRAKE, P4 CONN_SRV_FOOT, P5 CONN_VCC, P6 CONN_STEP_STOP, P7 CONN_LED, P8 CONN_BAT_INT, P9 CONN_EP_UART, U1 MCP23017

Commit message: Before major layout change
Parts:
- added C2: 100nF, Capacitors_SMD:C_0402, symbol C_Small
- added U2: TMP101, TO_SOT_Packages_SMD:SOT-23-6_Handsoldering, symbol TMP10X
- P21: footprint Pin_Headers:Pin_Header_Straight_1x12_Pitch1.27mm -> Pin_Headers:Pin_Header_Straight_1x15_Pitch1.27mm; symbol CONN_01X12 -> CONN_01X15
Connections:
- net A0: now also P21.13 (P13); no longer P21.11 (P11)
- net EP_EN: now also U1.22 (GPA5); no longer U1.23 (GPA6)
- net FRAME_STOP: now also U1.27 (GPB2); no longer U1.28 (GPB3)
- net GND: now also P21.12 (P12), P21.15 (P15), C2.1, U2.2 (GND); no longer P21.7 (P7)
- net LED_EN: now also U1.28 (GPB3); no longer U1.22 (GPA5)
- net SCK/SRV_LOCK: now also P21.11 (P11); no longer P21.12 (P12)
- net SCL: now also U2.1 (SCL)
- net SDA: now also U2.6 (SDA)
- net STEP_DIR: now also U1.24 (GPA7); no longer U1.25 (GPB0)
- net STEP_STOP1: now also U1.25 (GPB0); no longer U1.26 (GPB1)
- net STEP_STOP2: now also U1.26 (GPB1); no longer U1.27 (GPB2)
- net VCC: now also C2.2, U2.4 (V+)
- net ~STEP_SLP: now also U1.23 (GPA6); no longer U1.24 (GPA7)
- new net A6: P21.14 (P14), U2.3 (ALERT/ADD1)
- no-connect marks 2 -> 4
Other:
- moved on the sheet: P6, P9
Changed lines of the file:
@@
 Comment4 ""
 $EndDescr
-Text Label 12550 2850 2    60   ~ 0
+Text Label 12550 2700 2    60   ~ 0
 SRV_CAM
-Text Label 12550 3050 2    60   ~ 0
+Text Label 12550 2900 2    60   ~ 0
 MISO/SRV_BRAKE
-Text Label 12550 3250 2    60   ~ 0
+Text Label 12550 3000 2    60   ~ 0
 SCK/SRV_LOCK
-Text Label 12550 2950 2    60   ~ 0
+Text Label 12550 2800 2    60   ~ 0
 ~SS~/SRV_FOOT
 Text Label 12550 5000 2    60   ~ 0
@@
 SCL
 $Comp
-L CONN_01X12 P21
+L CONN_01X15 P21
 U 1 1 581029E7
 P 12750 2700
-F 0 "P21" H 12750 3400 50  0000 C CNN
+F 0 "P21" H 12750 3500 50  0000 C CNN
 F 1 "CONN1" V 12850 2750 50  0000 C CNN
-F 2 "Pin_Headers:Pin_Header_Straight_1x12_Pitch1.27mm" H 12750 2700 50  0001 C CNN
+F 2 "Pin_Headers:Pin_Header_Straight_1x15_Pitch1.27mm" H 12750 2700 50  0001 C CNN
 F 3 "" H 12750 2700 50  0000 C CNN
 	1    12750 2700
 	1    0    0    -1
 $EndComp
-Text Label 11200 2350 0    60   ~ 0
+Text Label 11200 2200 0    60   ~ 0
 FRAME_STOP
 Text Label 12550 4100 2    60   ~ 0
@@
 Text Label 12500 6300 2    60   ~ 0
 EP_VCC
-Text Label 12550 2150 2    60   ~ 0
+Text Label 12550 2000 2    60   ~ 0
 EP_RXD
-Text Label 12550 2450 2    60   ~ 0
+Text Label 12550 2300 2    60   ~ 0
 EP_TXD
 Text Label 9150 6450 0    60   ~ 0
@@
 Text Label 12500 7050 2    60   ~ 0
 EP_EN
-Text Label 12550 2350 2    60   ~ 0
+Text Label 12550 2200 2    60   ~ 0
 UART_RX
-Text Label 12550 2250 2    60   ~ 0
+Text Label 12550 2100 2    60   ~ 0
 UART_TX
 Text Label 9150 1700 0    60   ~ 0
@@
 Text Label 12500 6000 2    60   ~ 0
 GND
-Text Label 12550 3150 2    60   ~ 0
+Text Label 12550 3200 2    60   ~ 0
 A0
 Text Label 12500 6950 2    60   ~ 0
@@
 L CONN_01X04 P9
 U 1 1 581030F3
-P 11000 2300
-F 0 "P9" H 11000 2050 50  0000 C CNN
-F 1 "CONN_EP_UART" H 11350 2300 50  0000 C CNN
-F 2 "Connectors_Molex:Molex_PicoBlade_53047-0410" H 11000 2300 50  0001 C CNN
-F 3 "" H 11000 2300 50  0000 C CNN
-	1    11000 2300
+P 11000 2150
+F 0 "P9" H 11000 1900 50  0000 C CNN
+F 1 "CONN_EP_UART" H 11350 2150 50  0000 C CNN
+F 2 "Connectors_Molex:Molex_PicoBlade_53047-0410" H 11000 2150 50  0001 C CNN
+F 3 "" H 11000 2150 50  0000 C CNN
+	1    11000 2150
 	-1   0    0    1
 $EndComp
@@
 L GND #PWR02
 U 1 1 581031DD
-P 11200 2450
-F 0 "#PWR02" H 11200 2200 50  0001 C CNN
-F 1 "GND" H 11200 2300 50  0001 C CNN
-F 2 "" H 11200 2450 50  0000 C CNN
-F 3 "" H 11200 2450 50  0000 C CNN
-	1    11200 2450
+P 11200 2300
+F 0 "#PWR02" H 11200 2050 50  0001 C CNN
+F 1 "GND" H 11200 2150 50  0001 C CNN
+F 2 "" H 11200 2300 50  0000 C CNN
+F 3 "" H 11200 2300 50  0000 C CNN
+	1    11200 2300
 	1    0    0    -1
 $EndComp
@@
 L CONN_01X03 P6
 U 1 1 581067C5
-P 3800 2000
-F 0 "P6" H 3950 2000 50  0000 C CNN
-F 1 "CONN_STEP_STOP" H 3800 1800 50  0000 C CNN
-F 2 "Connectors_Molex:Molex_PicoBlade_53047-0310" H 3800 2000 50  0001 C CNN
-F 3 "" H 3800 2000 50  0000 C CNN
-	1    3800 2000
+P 3800 1900
+F 0 "P6" H 3950 1900 50  0000 C CNN
+F 1 "CONN_STEP_STOP" H 3800 1700 50  0000 C CNN
+F 2 "Connectors_Molex:Molex_PicoBlade_53047-0310" H 3800 1900 50  0001 C CNN
+F 3 "" H 3800 1900 50  0000 C CNN
+	1    3800 1900
 	-1   0    0    1
 $EndComp
@@
 L GND #PWR010
 U 1 1 58106AF4
-P 4000 2100
-F 0 "#PWR010" H 4000 1850 50  0001 C CNN
-F 1 "GND" H 4000 1950 50  0001 C CNN
-F 2 "" H 4000 2100 50  0000 C CNN
-F 3 "" H 4000 2100 50  0000 C CNN
-	1    4000 2100
+P 4000 2000
+F 0 "#PWR010" H 4000 1750 50  0001 C CNN
+F 1 "GND" H 4000 1850 50  0001 C CNN
+F 2 "" H 4000 2000 50  0000 C CNN
+F 3 "" H 4000 2000 50  0000 C CNN
+	1    4000 2000
 	1    0    0    -1
 $EndComp
@@
 L PWR_FLAG #FLG011
 U 1 1 581079B4
-P 4700 5150
-F 0 "#FLG011" H 4700 5245 50  0001 C CNN
-F 1 "PWR_FLAG" H 4700 5330 50  0000 C CNN
-F 2 "" H 4700 5150 50  0000 C CNN
-F 3 "" H 4700 5150 50  0000 C CNN
-	1    4700 5150
+P 2200 1450
+F 0 "#FLG011" H 2200 1545 50  0001 C CNN
+F 1 "PWR_FLAG" H 2200 1630 50  0000 C CNN
+F 2 "" H 2200 1450 50  0000 C CNN
+F 3 "" H 2200 1450 50  0000 C CNN
+	1    2200 1450
 	1    0    0    -1
 $EndComp
@@
 L GND #PWR012
 U 1 1 58107A60
-P 4700 5150
-F 0 "#PWR012" H 4700 4900 50  0001 C CNN
-F 1 "GND" H 4700 5000 50  0001 C CNN
-F 2 "" H 4700 5150 50  0000 C CNN
-F 3 "" H 4700 5150 50  0000 C CNN
-	1    4700 5150
+P 2200 1450
+F 0 "#PWR012" H 2200 1200 50  0001 C CNN
+F 1 "GND" H 2200 1300 50  0001 C CNN
+F 2 "" H 2200 1450 50  0000 C CNN
+F 3 "" H 2200 1450 50  0000 C CNN
+	1    2200 1450
 	1    0    0    -1
 $EndComp
@@
 L VCC #PWR013
 U 1 1 5815B14D
-P 4250 5150
-F 0 "#PWR013" H 4250 5000 50  0001 C CNN
-F 1 "VCC" H 4250 5300 50  0000 C CNN
-F 2 "" H 4250 5150 50  0000 C CNN
-F 3 "" H 4250 5150 50  0000 C CNN
-	1    4250 5150
+P 1750 1450
+F 0 "#PWR013" H 1750 1300 50  0001 C CNN
+F 1 "VCC" H 1750 1600 50  0000 C CNN
+F 2 "" H 1750 1450 50  0000 C CNN
+F 3 "" H 1750 1450 50  0000 C CNN
+	1    1750 1450
 	-1   0    0    1
 $EndComp
@@
 L PWR_FLAG #FLG014
 U 1 1 5815B27D
-P 4250 5150
-F 0 "#FLG014" H 4250 5245 50  0001 C CNN
-F 1 "PWR_FLAG" H 4250 5330 50  0000 C CNN
-F 2 "" H 4250 5150 50  0000 C CNN
-F 3 "" H 4250 5150 50  0000 C CNN
-	1    4250 5150
+P 1750 1450
+F 0 "#FLG014" H 1750 1545 50  0001 C CNN
+F 1 "PWR_FLAG" H 1750 1630 50  0000 C CNN
+F 2 "" H 1750 1450 50  0000 C CNN
+F 3 "" H 1750 1450 50  0000 C CNN
+	1    1750 1450
 	1    0    0    -1
 $EndComp
@@
 	1    0    0    -1
 $EndComp
+Text Label 4850 1900 2    60   ~ 0
+STEP_STOP1
 Text Label 4850 2000 2    60   ~ 0
-STEP_STOP1
+STEP_STOP2
 Text Label 4850 2100 2    60   ~ 0
-STEP_STOP2
-Text Label 4850 2200 2    60   ~ 0
 FRAME_STOP
 Text Label 4850 3000 2    60   ~ 0
@@
 Text Label 4850 2800 2    60   ~ 0
 FAN_TACHO
-Text Label 4850 1900 2    60   ~ 0
+Text Label 4850 3500 2    60   ~ 0
 STEP_DIR
-Text Label 4850 3500 2    60   ~ 0
+Text Label 4850 3400 2    60   ~ 0
 ~STEP_SLP
-Text Label 4850 3400 2    60   ~ 0
+Text Label 4850 3300 2    60   ~ 0
 EP_EN
-Text Label 4850 3300 2    60   ~ 0
+Text Label 4850 2200 2    60   ~ 0
 LED_EN
 $Comp
@@
 	1    0    0    -1
 $EndComp
-Text Label 12550 2550 2    60   ~ 0
+Text Label 12550 2400 2    60   ~ 0
 LED_EN
 $Comp
@@
 	-1   0    0    1
 $EndComp
-Text Label 12550 2650 2    60   ~ 0
+Text Label 12550 2500 2    60   ~ 0
 BAT_INT
 $Comp
@@
 	5950 1900 5850 1900
 Wire Wire Line
-	11200 2150 12550 2150
+	11200 2000 12550 2000
 Wire Wire Line
 	11200 5000 12550 5000
@@
 UART_RX
 Wire Wire Line
-	11200 2250 11850 2250
-Wire Wire Line
-	11850 2250 11850 2450
-Wire Wire Line
-	11850 2450 12550 2450
-Text Label 12550 2750 2    60   ~ 0
-GND
-NoConn ~ 12550 3150
+	11200 2100 11850 2100
+Wire Wire Line
+	11850 2100 11850 2300
+Wire Wire Line
+	11850 2300 12550 2300
+NoConn ~ 12550 3200
 Text Label 12550 3900 2    60   ~ 0
 SRV_VOUT
@@
 	11600 4600 12550 4600
 Wire Wire Line
-	4000 1900 4200 1900
-Wire Wire Line
-	4200 1900 4200 2000
-Wire Wire Line
-	4200 2000 4850 2000
-Wire Wire Line
-	4000 2000 4100 2000
-Wire Wire Line
-	4100 2000 4100 2100
-Wire Wire Line
-	4100 2100 4850 2100
+	4000 1800 4200 1800
+Wire Wire Line
+	4200 1800 4200 1900
+Wire Wire Line
+	4200 1900 4850 1900
+Wire Wire Line
+	4000 1900 4100 1900
+Wire Wire Line
+	4100 1900 4100 2000
+Wire Wire Line
+	4100 2000 4850 2000
+NoConn ~ 12550 2600
+Text Label 12550 3100 2    60   ~ 0
+GND
+Text Label 12550 3400 2    60   ~ 0
+GND
+Text Label 12550 3300 2    60   ~ 0
+A6
+$Comp
+L TMP10X U2
+U 1 1 581B96D8
+P 5150 4900
+F 0 "U2" H 4900 5150 60  0000 C CNN
+F 1 "TMP101" H 5450 4700 39  0000 C CNN
+F 2 "TO_SOT_Packages_SMD:SOT-23-6_Handsoldering" H 5200 4950 60  0001 C CNN
+F 3 "" H 5200 4950 60  0000 C CNN
+	1    5150 4900
+	1    0    0    -1
+$EndComp
+Text Label 4750 4800 2    60   ~ 0
+SCL
+Text Label 4750 4950 2    60   ~ 0
+SDA
+$Comp
+L GND #PWR024
+U 1 1 581BA498
+P 5150 5250
+F 0 "#PWR024" H 5150 5000 50  0001 C CNN
+F 1 "GND" H 5150 5100 50  0001 C CNN
+F 2 "" H 5150 5250 50  0000 C CNN
+F 3 "" H 5150 5250 50  0000 C CNN
+	1    5150 5250
+	1    0    0    -1
+$EndComp
+$Comp
+L VCC #PWR025
+U 1 1 581BA817
+P 5150 4450
+F 0 "#PWR025" H 5150 4300 50  0001 C CNN
+F 1 "VCC" H 5150 4600 50  0000 C CNN
+F 2 "" H 5150 4450 50  0000 C CNN
+F 3 "" H 5150 4450 50  0000 C CNN
+	1    5150 4450
+	1    0    0    -1
+$EndComp
+$Comp
+L C_Small C2
+U 1 1 581BAA92
+P 5500 4500
+F 0 "C2" V 5400 4550 50  0000 L CNN
+F 1 "100nF" V 5400 4250 50  0000 L CNN
+F 2 "Capacitors_SMD:C_0402" H 5500 4500 50  0001 C CNN
+F 3 "" H 5500 4500 50  0000 C CNN
+	1    5500 4500
+	0    1    1    0
+$EndComp
+Wire Wire Line
+	5150 4450 5150 4600
+Wire Wire Line
+	5150 4500 5400 4500
+Connection ~ 5150 4500
+Wire Wire Line
+	5150 5150 5150 5250
+Wire Wire Line
+	5150 5200 6000 5200
+Wire Wire Line
+	6000 5200 6000 4500
+Wire Wire Line
+	6000 4500 5600 4500
+Connection ~ 5150 5200
+NoConn ~ 5650 4950
+Text Label 5650 4800 0    60   ~ 0
+A6
 $EndSCHEMATC

Commit message: In progress, commit for backup
Parts:
- removed C1, C2: 100nF, Capacitors_SMD:C_0402, symbol C_Small
- removed P11: CONN_I2C, Connectors_Molex:Molex_PicoBlade_53047-0210, symbol CONN_01X02
- removed P18: CONN3, Pin_Headers:Pin_Header_Straight_1x10_Pitch1.27mm, symbol CONN_01X10
- removed P19: CONN4, Pin_Headers:Pin_Header_Straight_1x05_Pitch1.27mm, symbol CONN_01X05
- removed P21: CONN1, Pin_Headers:Pin_Header_Straight_1x15_Pitch1.27mm, symbol CONN_01X15
- removed P22: CONN2, Pin_Headers:Pin_Header_Straight_1x15_Pitch1.27mm, symbol CONN_01X15
- removed R1, R2: 10K, Resistors_SMD:R_0402_Handsoldering, symbol R_Small
- removed U1: MCP23017, Housings_DFN_QFN:QFN-28-1EP-NPTH_6x6mm_Pitch0.65mm, symbol MCP23017-QFN
- removed U2: TMP101, TO_SOT_Packages_SMD:SOT-23-6_Handsoldering, symbol TMP10X
- added P10: CONN_SPI0, Pin_Headers:Pin_Header_Straight_1x04_Pitch1.27mm, symbol CONN_01X04
- added P11: CONN_SPI1, Pin_Headers:Pin_Header_Straight_1x04_Pitch1.27mm, symbol CONN_01X04
- added P18: CONN2, Pin_Headers:Pin_Header_Straight_1x15_Pitch1.27mm, symbol CONN_01X15
- added P19: CONN_VCC, Socket_Strips:Socket_Strip_Straight_1x02, symbol CONN_01X02
- added P20: CONN1, Pin_Headers:Pin_Header_Straight_1x12_Pitch1.27mm, symbol CONN_01X12
- added P21: CONN3, Socket_Strips:Socket_Strip_Straight_1x06_Pitch1.27mm, symbol CONN_01X06
- added P22: CONN4, Socket_Strips:Socket_Strip_Straight_1x09_Pitch1.27mm, symbol CONN_01X09
- added P23: CONN_I2C0, Pin_Headers:Pin_Header_Straight_1x02_Pitch1.27mm, symbol CONN_01X02
- added P24: CONN_I2C1, Pin_Headers:Pin_Header_Straight_1x02_Pitch1.27mm, symbol CONN_01X02
- added TP1, TP4, TP7, TP8: TEST_1P, Pin_Headers:Pin_Header_Straight_1x01_Pitch1.27mm, symbol TEST_1P
- P1: renamed from P10; footprint Connectors_Molex:Molex_PicoBlade_53047-0410 -> Connectors_Molex:Molex_PicoBlade_53047-0510_DoubleSide; symbol CONN_01X04 -> CONN_01X05
- P12: renamed from P17; footprint Connectors_Molex:Molex_PicoBlade_53047-0510 -> Connectors_Molex:Molex_PicoBlade_53047-0210_DoubleSide; symbol CONN_01X05 -> CONN_01X02
- P13: renamed from P7; footprint Connectors_Molex:Molex_PicoBlade_53047-0410 -> Connectors_Molex:Molex_PicoBlade_53047-0410_DoubleSide
- P14: renamed from P5; footprint Connectors_Molex:Molex_PicoBlade_53047-0410 -> Connectors_Molex:Molex_PicoBlade_53047-0410_DoubleSide
- P15, P9: footprint Connectors_Molex:Molex_PicoBlade_53047-0410 -> Connectors_Molex:Molex_PicoBlade_53047-0410_DoubleSide
- P16: footprint Connectors_Molex:Molex_PicoBlade_53047-0210 -> Connectors_Molex:Molex_PicoBlade_53047-0410_DoubleSide; symbol CONN_01X02 -> CONN_01X04
- P17: renamed from P14; footprint Connectors_Molex:Molex_PicoBlade_53047-0410 -> Connectors_Molex:Molex_PicoBlade_53047-0410_DoubleSide
- P2: renamed from P1; footprint Connectors_Molex:Molex_PicoBlade_53047-0310 -> Connectors_Molex:Molex_PicoBlade_53047-0310_DoubleSide
- P3: renamed from P2; footprint Connectors_Molex:Molex_PicoBlade_53047-0310 -> Connectors_Molex:Molex_PicoBlade_53047-0310_DoubleSide
- P4: renamed from P3; footprint Connectors_Molex:Molex_PicoBlade_53047-0310 -> Connectors_Molex:Molex_PicoBlade_53047-0310_DoubleSide
- P5: renamed from P4; footprint Connectors_Molex:Molex_PicoBlade_53047-0310 -> Connectors_Molex:Molex_PicoBlade_53047-0310_DoubleSide
- P6: footprint Connectors_Molex:Molex_PicoBlade_53047-0310 -> Connectors_Molex:Molex_PicoBlade_53047-0310_DoubleSide
- P7: renamed from P12; footprint Connectors_Molex:Molex_PicoBlade_53047-0410 -> Connectors_Molex:Molex_PicoBlade_53047-0410_DoubleSide
- P8: footprint Connectors_Molex:Molex_PicoBlade_53047-0210 -> Connectors_Molex:Molex_PicoBlade_53047-0210_DoubleSide
- R1: renamed from R3; footprint Resistors_SMD:R_0402_Handsoldering -> Resistors_SMD:R_0402
Connections:
- net BTN2 is gone; now on net GND: P12.2 (P2)
- net BAT_INT: now also P22.5 (P5)
- net EP_RXD: now also P20.1 (P1)
- net EP_TXD: now also P20.3 (P3)
- net EP_VCC: now also P16.2 (P2), P21.5 (P5), P21.6 (P6)
- net FAN_TACHO: now also P18.6 (P6)
- net FAN_VOUT: now also P18.5 (P5)
- net GND: now also P1.1 (P1), P13.2 (P2), P16.3 (P3), P16.4 (P4), P19.1 (P1); no longer P1.2 (P2), P12.5 (P5), P13.1 (P1), P16.2 (P2)
- net IR_RX: now also P17.3 (P3), P22.6 (P6); no longer P17.1 (P1)
- net IR_TX: now also P22.4 (P4)
- net LED_CLK: now also P13.3 (P3), P18.14 (P14); no longer P13.4 (P4)
- net LED_DAT: now also P13.4 (P4), P18.13 (P13); no longer P13.3 (P3)
- net LED_VOUT: now also P13.1 (P1), P18.15 (P15); no longer P13.2 (P2)
- net SRV_CAM: now also P20.5 (P5)
- net SRV_VOUT: now also P20.9 (P9)
- net STEP_A1: now also P21.1 (P1)
- net STEP_A2: now also P21.2 (P2)
- net STEP_B1: now also P21.4 (P4)
- net STEP_B2: now also P21.3 (P3)
- net UART_RX: now also P20.4 (P4)
- net UART_TX: now also R1.2, P20.2 (P2); no longer R1.1
- net UART_VCC: now also P1.2 (P2), R1.1; no longer P1.1 (P1), R1.2
- net VCC: now also P17.1 (P1), P19.2 (P2); no longer P17.3 (P3)
- net BTN1 renamed BUTTON
- net BUTTON: now also P18.11 (P11)
- removed net BTN3: P12.3 (P3)
- removed net BTN4: P12.4 (P4)
- net FRAME_STOP renamed SCK0/FRAME_STOP
- net SCK0/FRAME_STOP: now also P10.1 (P1), P20.12 (P12)
- net MISO/SRV_BRAKE renamed SRV_BRAKE
- net SRV_BRAKE: now also P20.7 (P7)
- net MOSI/FAN_PWM renamed FAN_PWM
- net FAN_PWM: now also P18.7 (P7)
- net SCK/SRV_LOCK renamed SRV_LOCK
- net SRV_LOCK: now also P20.8 (P8)
- net STEP_STOP1 renamed MISO0/STEP_STOP2
- net MISO0/STEP_STOP2: now also P10.2 (P2), P20.11 (P11)
- net STEP_STOP2 renamed MOSI0/STEP_STOP1
- net MOSI0/STEP_STOP1: now also P10.3 (P3), P20.10 (P10)
- net ~SS~/SRV_FOOT renamed SRV_FOOT
- net SRV_FOOT: now also P20.6 (P6)
- new net A2: P18.12 (P12), TP4.1
- new net BAT2_CTL/SCK1: P11.2 (P2), P18.3 (P3)
- new net CHG2_CTL/MOSI1: P11.3 (P3), P18.2 (P2)
- new net CHG2_STAT/MISO1: P11.4 (P4), P18.1 (P1)
- new net HOST_INT: P1.5 (P5), P22.8 (P8)
- new net PWR_INT: P22.7 (P7), TP7.1
- new net SCL0: P18.9 (P9), P23.2 (P2)
- new net SCL1: P22.2 (P2), P24.2 (P2)
- new net SDA0: P18.10 (P10), P23.1 (P1)
- new net SDA1: P22.1 (P1), P24.1 (P1)
- new net TMP_INT0: P18.4 (P4), TP1.1
- new net TMP_INT1: P22.9 (P9), TP8.1
- new net ~RESET0: P10.4 (P4), P18.8 (P8)
- new net ~RESET1: P11.1 (P1), P22.3 (P3)
- no-connect marks 4 -> 0
Other:
- moved on the sheet: P13, P14, P15, P17, P2, P3, P4, P5, P6, P7, P8, P9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

Commit message: Major modification of body board and companions
Parts:
- removed TP1, TP7, TP8: TEST_1P, Pin_Headers:Pin_Header_Straight_1x01_Pitch1.27mm, symbol TEST_1P
- added P25: CONN_I2C2, Pin_Headers:Pin_Header_Straight_1x02_Pitch1.27mm, symbol CONN_01X02
- added P26: CONN_TMP, Connectors_Molex:Molex_PicoBlade_53047-0510_DoubleSide, symbol CONN_01X05
- P18: footprint Pin_Headers:Pin_Header_Straight_1x15_Pitch1.27mm -> Socket_Strips:Socket_Strip_Straight_1x15_Pitch1.27mm
- P20: footprint Pin_Headers:Pin_Header_Straight_1x12_Pitch1.27mm -> Socket_Strips:Socket_Strip_Straight_1x13_Pitch1.27mm; symbol CONN_01X12 -> CONN_01X13
- P24: footprint Pin_Headers:Pin_Header_Straight_1x02_Pitch1.27mm -> Connectors_Molex:Molex_PicoBlade_53047-0210_DoubleSide
Connections:
- net TMP_INT0 is gone; now on net FAN_VOUT: P18.4 (P4)
- net TMP_INT1 is gone; now on net SCL0: P22.9 (P9)
- net A2: now also P20.9 (P9); no longer P18.12 (P12)
- net BAT_INT: now also P22.7 (P7); no longer P22.5 (P5)
- net BUTTON: now also P18.12 (P12); no longer P18.11 (P11)
- net FAN_PWM: now also P18.6 (P6); no longer P18.7 (P7)
- net FAN_TACHO: now also P18.8 (P8); no longer P18.6 (P6)
- net FAN_VOUT: no longer P18.5 (P5)
- net GND: now also P26.1 (P1)
- net HOST_INT: now also P18.7 (P7); no longer P22.8 (P8)
- net IR_TX: now also P22.5 (P5); no longer P22.4 (P4)
- net MISO0/STEP_STOP2: now also P20.12 (P12); no longer P20.11 (P11)
- net MOSI0/STEP_STOP1: now also P20.11 (P11); no longer P20.10 (P10)
- net PWR_INT: now also P22.1 (P1); no longer P22.7 (P7)
- net SCK0/FRAME_STOP: now also P20.13 (P13); no longer P20.12 (P12)
- net SCL0: now also P18.10 (P10), P25.2 (P2); no longer P18.9 (P9)
- net SCL1: now also P22.3 (P3), P26.3 (P3); no longer P22.2 (P2)
- net SDA0: now also P18.11 (P11), P22.8 (P8), P25.1 (P1); no longer P18.10 (P10)
- net SDA1: now also P22.2 (P2), P26.4 (P4); no longer P22.1 (P1)
- net SRV_VOUT: now also P20.10 (P10); no longer P20.9 (P9)
- net VCC: now also P26.5 (P5)
- net ~RESET0: now also P18.9 (P9); no longer P18.8 (P8)
- net ~RESET1: now also P22.4 (P4); no longer P22.3 (P3)
- new net TMP_INT: P18.5 (P5), P26.2 (P2)
- no-connect marks 0 -> 1
Other:
- moved on the sheet: P1, P10, P11, P12, P13, P14, P15, P16, P17, P18, P19, P2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
