File: subs/body/pwr/pwr.sch (KiCad schematic (older format))
At the start: 2 parts, among them P1 CON_BAT_IN, P2 CON_BAT_OUT

Commit message: In progress, commit for backup
Parts:
- removed P1: CON_BAT_IN, Socket_Strips:Socket_Strip_Straight_2x05, symbol CONN_02X05
- removed P2: CON_BAT_OUT, Socket_Strips:Socket_Strip_Straight_2x04, symbol CONN_02X04
- added C? (x3): 470uF, symbol CP1_Small
- added P?: CONN4, Pin_Headers:Pin_Header_Straight_1x09_Pitch1.27mm, symbol CONN_01X09
- added P?: CONN_VCC, Pin_Headers:Pin_Header_Straight_1x02, symbol CONN_01X02
- added P?: CONN5, Pin_Headers:Pin_Header_Straight_2x05, symbol CONN_02X05
- added P?: USB_A, symbol USB_A
- added P? (x2): CONN_01X03, symbol CONN_01X03
- added P?: CONN_CHG, Pin_Headers:Pin_Header_Straight_1x02, symbol CONN_01X03
- added R?: 2M, symbol R_Small
- added R?: 3M, symbol R_Small
- added R?: 4.42M, symbol R_Small
- added R?: 604K, symbol R_Small
- added U?: TPS61800 module, Converters_DCDC_ACDC:DCDC_Conv_TPS61800-Boost, symbol DCDC_Module
- added U?: G5177 module, Converters_DCDC_ACDC:DCDC_Conv_G5177-Boost, symbol DCDC_Module
- added U?: 100W module, Converters_DCDC_ACDC:DCDC_Conv_100W-Boost, symbol DCDC_Module
- added U?: 1S 4A/8A Charger, Converters_DCDC_ACDC:DCDC_Charger-1S-4A-8A-Bucket, symbol DCDC_Module
- added U?: HG6293 Charger, Converters_DCDC_ACDC:DCDC_Conv_100W-Boost, symbol DCDC_Module
Connections:
- net BAT: now also C?.1, P?.3 (P3), P?.4 (P4), P?.5 (P5), P?.6 (P6), U?.2 (VIN), U?.2 (VIN), U?.2 (VIN)
- net CHARGE: now also P?.7 (P7), P?.8 (P8), U?.3 (VOUT), U?.3 (VOUT)
- net GND: now also C?.2, C?.2, C?.2, P?.1 (P1), P?.1 (P1), P?.1 (P1), P?.10 (P10), P?.2 (P2), P?.4 (GND), P?.5 (shield), P?.9 (P9), R?.2, R?.2, U?.1 (GND), U?.1 (GND), U?.1 (GND), U?.1 (GND), U?.1 (GND)
- new net: P?.2 (D-), P?.2 (P2)
- new net: P?.2 (P2), P?.3 (D+)
- new net BAT_INT: P?.5 (P5)
- new net CHG_IN: C?.1, P?.1 (VBUS), P?.2 (P2), U?.2 (VIN), U?.2 (VIN)
- new net HOST_INT: P?.8 (P8)
- new net IR_RX: P?.6 (P6)
- new net IR_TX: P?.4 (P4)
- new net PWR_INT: P?.7 (P7)
- new net SCL1: P?.2 (P2)
- new net SDA1: P?.1 (P1)
- new net TMP_INT1: P?.9 (P9)
- new net V0.6: P?.3 (P3), P?.3 (P3), R?.1, R?.2
- new net V3.3: P?.1 (P1), P?.1 (P1), R?.1, R?.2
- new net VCC: C?.1, P?.2 (P2), P?.3 (P3), R?.1, R?.1, U?.3 (VOUT), U?.3 (VOUT), U?.3 (VOUT)
- new net ~RESET1: P?.3 (P3)
Other:
- note added: "QC2.0 high voltage request for 12V input with D+D- \nboth 0.6V, and 9V with D+ 3.3V and D- 0.6V."

Commit message: Major modification of body board and companions
Parts:
- removed P?: CONN4, Pin_Headers:Pin_Header_Straight_1x09_Pitch1.27mm, symbol CONN_01X09
- removed P?: USB_A, symbol USB_A
- removed P? (x2): CONN_01X03, symbol CONN_01X03
- removed P?: CONN_CHG, Pin_Headers:Pin_Header_Straight_1x02, symbol CONN_01X03
- removed R?: 2M, symbol R_Small
- removed R?: 3M, symbol R_Small
- removed R?: 4.42M, symbol R_Small
- removed R?: 604K, symbol R_Small
- removed U?: 100W module, Converters_DCDC_ACDC:DCDC_Conv_100W-Boost, symbol DCDC_Module
- removed U?: HG6293 Charger, Converters_DCDC_ACDC:DCDC_Conv_100W-Boost, symbol DCDC_Module
- added C4, C5, C6: 47uF, Capacitors_SMD:C_1206, symbol C_Small
- added P2: USB_Micro, Connect:USB_Micro-B, symbol USB_OTG
- added P4, P5: CONN_01X03, Pin_Headers:Pin_Header_Straight_1x03_Pitch1.27mm, symbol CONN_01X03
- added P6, P7, P8: CONN_01X01, Pin_Headers:Pin_Header_Straight_1x01, symbol CONN_01X01
- added R1: 2M, Resistors_SMD:R_0402, symbol R_Small
- added R2: 1M, Resistors_SMD:R_0402, symbol R_Small
- added R3: 400K, Resistors_SMD:R_0402, symbol R_Small
- added U4: LDO_3V5, Converters_DCDC_ACDC:LDO_RT9018, symbol LDO_Module
- C1, C2, C3: renamed from C?; value 470uF -> 47uF; footprint (none) -> Capacitors_SMD:C_1206; symbol CP1_Small -> C_Small
- P1: renamed from P?; footprint Pin_Headers:Pin_Header_Straight_2x05 -> Socket_Strips:Socket_Strip_Straight_2x05
- P3: renamed from P?; footprint Pin_Headers:Pin_Header_Straight_1x02 -> Socket_Strips:Socket_Strip_Straight_1x02
- U5: renamed from U?; value 1S 4A/8A Charger -> TP5000 Charger; footprint Converters_DCDC_ACDC:DCDC_Charger-1S-4A-8A-Bucket -> Converters_DCDC_ACDC:DCDC_Charger-TP5000-Bucket
- gave numbers to parts that had none: 2
Connections:
- net BAT: now also C5.1, P7.1 (P1), U4.2 (VIN)
- net CHG_IN: now also C4.1, P2.1 (VBUS), P8.1 (P1)
- net GND: now also C4.2, C5.2, C6.2, P2.5 (GND), P2.6 (shield), P6.1 (P1), R3.2, U4.1 (GND)
- net V0.6: now also P2.2 (D-), P4.1 (P1), P4.2 (P2), P5.1 (P1), R2.2, R3.1
- net V3.3: now also P2.3 (D+), P4.3 (P3), P5.2 (P2), P5.3 (P3), R1.2, R2.1
- net VCC: now also C6.1, R1.1, U4.3 (VCC)
- no-connect marks 0 -> 1
Other:
- moved on the sheet: P1, P3, U1, U2, U5
